File: Hardware Design/esp32 master.kicad_sch (KiCad schematic)
At the start: 26 parts, among them J1 Barrel_Jack_PTH, J2 Conn_01x06_Socket, J3 Conn_01x05_Socket, J5 Conn_01x04_Socket, J6 Conn_01x04_Socket, U1 LM2596S-5, U2 ESP32-DevKitC

Commit message: Refactor code structure for improved readability and maintainability
Parts:
- removed JP1: ~, Jumper:SolderJumper-2_P1.3mm_Open_RoundedPad1.0x1.5mm, symbol SparkFun-Jumper:SolderJumper_2_Open
- added D4, D5: SD36_SOD323, Diode_SMD:D_SOD-323, symbol Diode:SD36_SOD323
- added J4: Conn_01x02_Socket, Connector_PinHeader_2.54mm:PinHeader_1x02_P2.54mm_Vertical, symbol Connector:Conn_01x02_Socket
- added R4, R5: 10k, SparkFun-Resistor:R_0603_1608Metric, symbol SparkFun-Resistor:10k_0603
Connections:
- net 3v3: now also D5.2 (A2)
- net 5V: now also D4.2 (A2), R5.2
- net GND: now also D4.1 (A1), D5.1 (A1), R4.1
- net STBY: now also R5.1
- net Servo1: now also R4.2
- net at C2.1, C4.1, Driver1.1 (VM)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: now also J4.2 (Pin_2)
- net at R1.2, R2.1: now also J4.1 (Pin_1)
Other:
- moved on the sheet: R1, R2

Commit message: Refactor code structure for improved readability and maintainability
Other:
- note added: "ESP32 Dev Kit"
- note added: "Motor Drivers"
- title: esp32 master -> Break-out Board for the RobotCar
- moved on the sheet: C1, C2, C3, C4, C5, C6, D1, D2, D3, D4, D5, Driver1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

Commit message: Refactor code structure for improved readability and maintainability
Parts:
- removed D4, D5: SD36_SOD323, Diode_SMD:D_SOD-323, symbol Diode:SD36_SOD323
- removed R1: 4.7k, PCM_Resistor_THT_US_AKL:R_Axial_DIN0207_L6.3mm_D2.5mm_P7.62mm_Horizontal, symbol PCM_Resistor_US_AKL:R_DIN0207_P7.62mm
- removed R2: 10k, PCM_Resistor_THT_US_AKL:R_Axial_DIN0207_L6.3mm_D2.5mm_P7.62mm_Horizontal, symbol PCM_Resistor_US_AKL:R_DIN0207_P7.62mm
- removed U2: ESP32-DevKitC, PCM_Espressif:ESP32-DevKitC, symbol PCM_Espressif:ESP32-DevKitC
- added C11: 10uF, PCM_JLCPCB:C_0603, symbol PCM_JLCPCB-Capacitors:0603,10uF
- added C7, C8, C9: 0.1uF, SparkFun-Capacitor:C_0402_1005Metric, symbol SparkFun-Capacitor:0.1uF_0402_16V_10%
- added Q1, Q2: BC817-25-TP, digikey-footprints:SOT-23-3, symbol dk_Transistors-Bipolar-BJT-Single:BC817-25-TP
- added R1, R2, R6: 10k, SparkFun-Resistor:R_0603_1608Metric, symbol SparkFun-Resistor:10k_0603
- added R7, R8: 0, SparkFun-Resistor:R_0603_1608Metric, symbol SparkFun-Resistor:0_0603
- added ST4: Standoff, SparkFun-Hardware:Standoff, symbol SparkFun-Hardware:Standoff
- added SW1, SW2: SMD_5.2x5.2mm_h1.9mm, SparkFun-Switch:Push_SMD_5.2x5.2mm_h1.9mm, symbol SparkFun-Switch:SPST_Push_SMD_5.2x5.2mm_h1.9mm
- added U2: ESP32-WROOM-32D, RF_Module:ESP32-WROOM-32D, symbol RF_Module:ESP32-WROOM-32D
- C1: footprint PCM_Capacitor_THT_AKL:CP_Radial_D8.0mm_P3.50mm -> Capacitor_THT:CP_Radial_D8.0mm_P2.50mm
- C2, C4: footprint Capacitor_THT:C_Radial_D5.0mm_H5.0mm_P2.00mm -> Capacitor_THT:C_Radial_D6.3mm_H7.0mm_P2.50mm
- C3, C6: footprint Capacitor_THT:C_Disc_D3.0mm_W1.6mm_P2.50mm -> Capacitor_SMD:C_0805_2012Metric_Pad1.18x1.45mm_HandSolder
- C5: footprint PCM_Capacitor_THT_AKL:CP_Radial_D8.0mm_P3.50mm -> Capacitor_SMD:CP_Elec_6.3x5.4_Nichicon
- D3: footprint LED_THT:LED_D3.0mm -> LED_SMD:LED_0603_1608Metric_Pad1.05x0.95mm_HandSolder
- Driver1, Driver2: footprint tb6612fng:tb6612fng breakout board -> tb6612fng:DIP-16_591_ELL
- J5: footprint Connector_PinHeader_2.00mm:PinHeader_1x04_P2.00mm_Vertical -> Connector_PinHeader_2.54mm:PinHeader_1x04_P2.54mm_Vertical
- J6: footprint Connector_PinHeader_2.00mm:PinHeader_1x04_P2.00mm_Vertical -> Connector_JST:JST_EH_B4B-EH-A_1x04_P2.50mm_Vertical
- R3: footprint Resistor_THT:R_Axial_DIN0207_L6.3mm_D2.5mm_P2.54mm_Vertical -> Resistor_SMD:R_0805_2012Metric_Pad1.20x1.40mm_HandSolder
Connections:
- net 3v3: now also C11.1, C8.1, R1.2, U2.2 (VDD)
- net GND: now also C11.2, C7.2, C8.2, C9.2, SW1.1, SW2.2, U2.1 (GND), U2.15 (GND), U2.38 (GND), U2.39 (GND)
- net VM: now also J4.1 (Pin_1)
- net AIN1 renamed MOTOR1_AIN1
- net AIN12 renamed MOTOR2_AIN1
- net AIN2 renamed MOTOR1_AIN2
- net AIN22 renamed MOTOR2_AIN2
- net BIN1 renamed MOTOR1_BIN1
- net BIN12 renamed MOTOR2_BIN1
- net BIN2 renamed MOTOR1_BIN2
- net BIN22 renamed MOTOR2_BIN2
- net PWMA renamed MOTOR1_PWMA
- net PWMA2 renamed MOTOR2_PWMA
- net PWMB renamed MOTOR1_PWMB 
- net PWMB2 renamed MOTOR2_PWMB
- net STBY renamed STBY_PIN
- new net: Q1.1 (B), R2.1
- new net: Q2.1 (B), R6.1
- new net DTR: Q2.3 (C), R2.2
- new net EN: C9.1, Q1.3 (C), R1.1, SW1.2, U2.3 (EN)
- new net IO0: C7.1, Q2.2 (E), SW2.1, U2.25 (IO0)
- new net IO12: U2.14 (IO12)
- new net IO13: U2.16 (IO13)
- new net IO14: U2.13 (IO14)
- new net IO15: U2.23 (IO15)
- new net IO16: U2.27 (IO16)
- new net IO17: U2.28 (IO17)
- new net IO18: U2.30 (IO18)
- new net IO19: U2.31 (IO19)
- new net IO2: U2.24 (IO2)
- new net IO21: U2.33 (IO21)
- new net IO22: U2.36 (IO22)
- new net IO23: U2.37 (IO23)
- new net IO25: U2.10 (IO25)
- new net IO26: U2.11 (IO26)
- new net IO27: U2.12 (IO27)
- new net IO32: U2.8 (IO32)
- new net IO33: U2.9 (IO33)
- new net IO34: U2.6 (IO34)
- new net IO35: U2.7 (IO35)
- new net IO4: U2.26 (IO4)
- new net IO5: U2.29 (IO5)
- new net RTS: Q1.2 (E), R6.2
- new net RX: R8.2, U2.34 (RXD0/IO3)
- new net RXD: R8.1
- new net SENSOR_VN: U2.5 (SENSOR_VN)
- new net SENSOR_VP: U2.4 (SENSOR_VP)
- new net TX: R7.2, U2.35 (TXD0/IO1)
- new net TXD: R7.1
Other:
- note removed: "ESP32 Dev Kit"
- moved on the sheet: C2, C4, Driver1, Driver2, J2, J4, J5, J6, R4, R5
